Commit message: testing urdf file

File: assets/urdf/test.urdf (robot description, URDF)
Before this commit: robot caterpillar, 4 links, 3 joints
Links:
- added link intermediate_0_1, mass 0.001
- added link intermediate_1_2, mass 0.001
- added link intermediate_2_3, mass 0.001
Joints:
- removed joint joint_0_1
- removed joint joint_1_2
- removed joint joint_2_3
- added joint joint_0_1_pitch: type revolute, parent segment_0, child intermediate_0_1, origin xyz=0.03 0 0 rpy=0 0 0, axis 0 0 1, limit lower=-1.57 upper=1.57 effort=1.0 velocity=2.0
- added joint joint_0_1_yaw: type revolute, parent intermediate_0_1, child segment_1, origin xyz=0 0 0 rpy=0 0 0, axis 0 1 0, limit lower=-1.57 upper=1.57 effort=1.0 velocity=2.0
- added joint joint_1_2_pitch: type revolute, parent segment_1, child intermediate_1_2, origin xyz=0.06 0 0 rpy=0 0 0, axis 0 0 1, limit lower=-1.57 upper=1.57 effort=1.0 velocity=2.0
- added joint joint_1_2_yaw: type revolute, parent intermediate_1_2, child segment_2, origin xyz=0 0 0 rpy=0 0 0, axis 0 1 0, limit lower=-1.57 upper=1.57 effort=1.0 velocity=2.0
- added joint joint_2_3_pitch: type revolute, parent segment_2, child intermediate_2_3, origin xyz=0.06 0 0 rpy=0 0 0, axis 0 0 1, limit lower=-1.57 upper=1.57 effort=1.0 velocity=2.0
- added joint joint_2_3_yaw: type revolute, parent intermediate_2_3, child segment_3, origin xyz=0 0 0 rpy=0 0 0, axis 0 1 0, limit lower=-1.57 upper=1.57 effort=1.0 velocity=2.0

Commit message: Implement addLimb in evolve

File: assets/urdf/test.urdf (robot description, URDF)
Before this commit: robot caterpillar, 4 links, 3 joints
Links:
- removed link segment_0
- removed link segment_1
- removed link segment_2
- removed link segment_3
- added link segment_0_limb, mass 0.10; collision capsule length=0.06 radius=0.02; visual capsule length=0.06 radius=0.02
- added link segment_1_torso, mass 0.10; collision capsule length=0.06 radius=0.02; visual capsule length=0.06 radius=0.02
- added link segment_2_limb, mass 0.10; collision capsule length=0.06 radius=0.02; visual capsule length=0.06 radius=0.02
- added link segment_3_limb, mass 0.10; collision capsule length=0.06 radius=0.02; visual capsule length=0.06 radius=0.02

Commit message: Complete addLimb implementation

File: assets/urdf/test.urdf (robot description, URDF)
Before this commit: robot caterpillar, 4 links, 3 joints
Joints:
- joint joint_0_1: child segment_1 -> segment_1_torso; parent segment_0 -> segment_0_limb
- joint joint_1_2: child segment_2 -> segment_2_limb; parent segment_1 -> segment_1_torso
- joint joint_2_3: child segment_3 -> segment_3_limb; parent segment_2 -> segment_2_limb

Commit message: Implement evolve addLimb functionality (#14)
Co-authored-by: fjcu256 <106101347+fjcu256@users.noreply.github.com>
Co-authored-by: Krisi Hristova <kh3339@drexel.edu>

File: assets/urdf/test.urdf (robot description, URDF)
Before this commit: robot caterpillar, 4 links, 3 joints
Links:
- removed link segment_0
- removed link segment_1
- removed link segment_2
- removed link segment_3
- added link segment_0_limb, mass 0.10; collision capsule length=0.06 radius=0.02; visual capsule length=0.06 radius=0.02
- added link segment_1_torso, mass 0.10; collision capsule length=0.06 radius=0.02; visual capsule length=0.06 radius=0.02
- added link segment_2_limb, mass 0.10; collision capsule length=0.06 radius=0.02; visual capsule length=0.06 radius=0.02
- added link segment_3_limb, mass 0.10; collision capsule length=0.06 radius=0.02; visual capsule length=0.06 radius=0.02
Joints:
- joint joint_0_1: child segment_1 -> segment_1_torso; parent segment_0 -> segment_0_limb
- joint joint_1_2: child segment_2 -> segment_2_limb; parent segment_1 -> segment_1_torso
- joint joint_2_3: child segment_3 -> segment_3_limb; parent segment_2 -> segment_2_limb
