Commit message: add training implementation

File: assets/urdf/agents/caterpillar.urdf (robot description, URDF)
Before this commit: robot caterpillar, 4 links, 3 joints
Links:
- removed link segment_0_limb
- removed link segment_1_torso
- removed link segment_2_limb
- removed link segment_3_limb
- added link intermediate_0_1
- added link intermediate_1_2
- added link intermediate_2_3
- added link segment_1; collision capsule length=0.06 radius=0.02; visual capsule length=0.06 radius=0.02
- added link segment_2; collision capsule length=0.06 radius=0.02; visual capsule length=0.06 radius=0.02
- added link segment_3; collision capsule length=0.06 radius=0.02; visual capsule length=0.06 radius=0.02
- added link torso; collision capsule length=0.06 radius=0.02; visual capsule length=0.06 radius=0.02
Joints:
- added joint joint_2_3_yaw: type revolute, parent intermediate_2_3, child segment_3, origin xyz=0 0 0 rpy=0 0 0, axis 0 1 0, limit lower=-1.57 upper=1.57 effort=1.0 velocity=2.0
